File: productfiles/circuitboard/moko/moko.kicad_sch (KiCad schematic)
At the start: 5 parts, among them SW1 kbd_SW_PUSH

Commit message: update circuit diagram
Parts:
- removed J?: MJ-4PP-9, symbol moko-rescue:MJ-4PP-9-kbd
- removed J?: Conn_01x03, symbol Connector_Generic:Conn_01x03
- removed RSW?: SW_PUSH, symbol moko-rescue:SW_PUSH-kbd
- removed SW1: kbd_SW_PUSH, symbol moko-rescue:SW_PUSH-kbd
- added D1, D10, D11, D12, D13, D14, D15, D16, D17, D2, D3, D4, D5, D6, D7, D8, D9: D, mykeyboardparts:D3_SMD_rev, symbol Device:D
- added J1, J4: Conn_01x06, symbol Connector_Generic:Conn_01x06
- added J3: AudioJack4, mykeyboardparts:MJ-4PP-9_rev, symbol Connector_Audio:AudioJack4
- added RSW1: SW_Push, keyboard_parts.pretty-master:SW_TACT_TH_HORIZ, symbol Switch:SW_Push
- added SW1, SW10, SW11, SW12, SW13, SW14, SW15, SW2, SW3, SW4, SW5, SW6, SW7, SW8, SW9: SW_PUSH, symbol kbd:SW_PUSH
- added SW16, SW18: SW_Push, symbol Switch:SW_Push
- U1: renamed from U?; footprint (none) -> mykeyboardparts:ProMicro_v2; symbol moko-rescue:ProMicro-kbd -> kbd:ProMicro
Connections:
- net GND: now also J1.6 (Pin_6), J3.S, J4.6 (Pin_6), RSW1.2
- net LED: now also J1.4 (Pin_4), J3.R1
- net VCC: now also J1.1 (Pin_1), J3.T, J4.1 (Pin_1)
- net col0: now also SW10.1, SW15.1, SW5.1
- net col1: now also SW1.1, SW11.1, SW6.1
- net col2: now also SW12.1, SW2.1, SW7.1
- net col3: now also J1.2 (Pin_2), SW13.1, SW3.1, SW8.1
- net col4: now also J1.3 (Pin_3), SW14.1, SW4.1, SW9.1
- net data: now also J3.R2
- net reset: now also RSW1.1
- net row0: now also D1.1 (K), D2.1 (K), D3.1 (K), D4.1 (K)
- net row1: now also D5.1 (K), D6.1 (K), D7.1 (K), D8.1 (K), D9.1 (K)
- net row2: now also D10.1 (K), D11.1 (K), D12.1 (K), D13.1 (K), D14.1 (K)
- net row3: now also D15.1 (K), J1.5 (Pin_5)
- net col5: no longer names the net of U1.18 (F6)
- net row4: no longer names the net of U1.8 (C6)
- new net: D14.2 (A), SW14.2
- new net: D15.2 (A), SW15.2
- new net: D17.2 (A), SW16.2
- new net: D6.2 (A), SW6.2
- new net: D8.2 (A), SW8.2
- new net: D9.2 (A), SW9.2
- new net: D1.2 (A), SW1.2
- new net: D16.2 (A), SW18.2
- new net: D11.2 (A), SW11.2
- new net: D4.2 (A), SW4.2
- new net: D10.2 (A), SW10.2
- new net: D7.2 (A), SW7.2
- new net: D13.2 (A), SW13.2
- new net: D5.2 (A), SW5.2
- new net: D2.2 (A), SW2.2
- new net: D12.2 (A), SW12.2
- new net: D3.2 (A), SW3.2
- new net col3*: J4.2 (Pin_2), SW18.1
- new net col4*: J4.3 (Pin_3), SW16.1
- new net row3*: D16.1 (K), D17.1 (K), J4.5 (Pin_5)
- no-connect marks 4 -> 9

Commit message: update footprint
Parts:
- SW1, SW10, SW11, SW12, SW13, SW14, SW15, SW2, SW3, SW4, SW5, SW6, SW7, SW8, SW9: symbol kbd:SW_PUSH -> 0-kbd:SW_PUSH
- U1: footprint mykeyboardparts:ProMicro_v2 -> 0-mykeyboardparts:ProMicro_v2; symbol kbd:ProMicro -> 0-kbd:ProMicro
- renumbered J3 to J2, J4 to J3, SW18 to SW16, SW16 to SW17
Other:
- moved on the sheet: J2, RSW1

Commit message: create pcb data
Parts:
- D1, D10, D11, D12, D13, D14, D15, D16, D17, D2, D3, D4, D5, D6, D7, D8, D9: footprint mykeyboardparts:D3_SMD_rev -> 0-moko_Library:D3_SMD_rev
- J1, J3: footprint (none) -> 0-moko_Library:board_conector_6pin_th
- J2: footprint mykeyboardparts:MJ-4PP-9_rev -> 0-moko_Library:MJ-4PP-9_rev_2
- RSW1: footprint keyboard_parts.pretty-master:SW_TACT_TH_HORIZ -> 0-moko_Library:ResetSW_Anled_MJP1117
- SW1, SW10, SW11, SW12, SW13, SW14, SW15, SW2, SW3, SW4, SW5, SW6, SW7, SW8, SW9: value SW_PUSH -> SW_Push; footprint (none) -> 0-moko_Library:CherryMX_Choc_Hotswap; symbol 0-kbd:SW_PUSH -> Switch:SW_Push
- SW16, SW17: footprint (none) -> 0-moko_Library:CherryMX_Choc_Hotswap
- U1: footprint 0-mykeyboardparts:ProMicro_v2 -> 0-moko_Library:ProMicro_v2
Connections:
- net LED*: now reaches J3.4 (Pin_4)
- no-connect marks 9 -> 8
Other:
- moved on the sheet: D1, D10, D11, D12, D13, D14, D15, D2, D3, D4, D5, D6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
