File: productfiles/circuitboard/moko/moko.kicad_sch (KiCad schematic)
At the start: 39 parts, among them J1 Conn_01x06, J2 AudioJack4, J3 Conn_01x06, SW1 SW_Push, SW10 SW_Push, SW11 SW_Push, SW12 SW_Push, SW13 SW_Push, SW14 SW_Push, SW15 SW_Push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

Commit message: fix pcb and sch
Connections:
- net data: now also J2.R2
Changed lines of the file:
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@@
-	(wire
-		(pts
-			(xy 121.92 31.75) (xy 121.92 40.64)
-		)
-		(stroke
-			(width 0)
-			(type default)
-		)
-	)
 	(wire
 		(pts
@@
 		)
 		(stroke
+			(width 0)
+			(type default)
+		)
+	)
+	(wire
+		(pts
+			(xy 43.18 135.89) (xy 50.8 135.89)
+		)
+		(stroke

Commit message: board upd8
Parts:
- RSW1: footprint 0-moko_Library:ResetSW_Anled_MJP1117 -> 0-moko_Library:ResetSW
- SW1, SW10, SW11, SW12, SW13, SW14, SW15, SW16, SW17, SW2, SW3, SW4, SW5, SW6, SW7, SW8, SW9: footprint 0-moko_Library:CherryMX_Choc_Hotswap -> 0-moko_Library:CherryMX_Hotswap
- U1: footprint 0-moko_Library:ProMicro_v2 -> 0-moko_Library:ProMicro_rev_2
Changed lines of the file:
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@@
 			)
 		)
-		(property "Footprint" "0-moko_Library:ProMicro_v2"
+		(property "Footprint" "0-moko_Library:ProMicro_rev_2"
 			(at 55.626 68.834 0)
 			(effects
@@
 			)
 		)
-		(property "Footprint" "0-moko_Library:CherryMX_Choc_Hotswap"
+		(property "Footprint" "0-moko_Library:CherryMX_Hotswap"
 			(at 195.58 76.2 0)
 			(effects
@@
 			)
 		)
-		(property "Footprint" "0-moko_Library:CherryMX_Choc_Hotswap"
+		(property "Footprint" "0-moko_Library:CherryMX_Hotswap"
 			(at 104.14 96.52 0)
 			(effects
@@
 			)
 		)
-		(property "Footprint" "0-moko_Library:ResetSW_Anled_MJP1117"
+		(property "Footprint" "0-moko_Library:ResetSW"
 			(at 55.88 102.87 0)
 			(effects
@@
 			)
 		)
-		(property "Footprint" "0-moko_Library:CherryMX_Choc_Hotswap"
+		(property "Footprint" "0-moko_Library:CherryMX_Hotswap"
 			(at 172.72 55.88 0)
 			(effects
@@
 			)
 		)
-		(property "Footprint" "0-moko_Library:CherryMX_Choc_Hotswap"
+		(property "Footprint" "0-moko_Library:CherryMX_Hotswap"
 			(at 195.58 35.56 0)
 			(effects
@@
 			)
 		)
-		(property "Footprint" "0-moko_Library:CherryMX_Choc_Hotswap"
+		(property "Footprint" "0-moko_Library:CherryMX_Hotswap"
 			(at 127 76.2 0)
 			(effects
@@
 			)
 		)
-		(property "Footprint" "0-moko_Library:CherryMX_Choc_Hotswap"
+		(property "Footprint" "0-moko_Library:CherryMX_Hotswap"
 			(at 149.86 55.88 0)
 			(effects
@@
 			)
 		)
-		(property "Footprint" "0-moko_Library:CherryMX_Choc_Hotswap"
+		(property "Footprint" "0-moko_Library:CherryMX_Hotswap"
 			(at 195.58 55.88 0)
 			(effects
@@
 			)
 		)
-		(property "Footprint" "0-moko_Library:CherryMX_Choc_Hotswap"
+		(property "Footprint" "0-moko_Library:CherryMX_Hotswap"
 			(at 172.72 76.2 0)
 			(effects
@@
 			)
 		)
-		(property "Footprint" "0-moko_Library:CherryMX_Choc_Hotswap"
+		(property "Footprint" "0-moko_Library:CherryMX_Hotswap"
 			(at 127 55.88 0)
 			(effects
@@
 			)
 		)
-		(property "Footprint" "0-moko_Library:CherryMX_Choc_Hotswap"
+		(property "Footprint" "0-moko_Library:CherryMX_Hotswap"
 			(at 104.14 76.2 0)
 			(effects
@@
 			)
 		)
-		(property "Footprint" "0-moko_Library:CherryMX_Choc_Hotswap"
+		(property "Footprint" "0-moko_Library:CherryMX_Hotswap"
 			(at 149.86 35.56 0)
 			(effects
@@
 			)
 		)
-		(property "Footprint" "0-moko_Library:CherryMX_Choc_Hotswap"
+		(property "Footprint" "0-moko_Library:CherryMX_Hotswap"
 			(at 148.59 165.1 0)
 			(effects
@@
 			)
 		)
-		(property "Footprint" "0-moko_Library:CherryMX_Choc_Hotswap"
+		(property "Footprint" "0-moko_Library:CherryMX_Hotswap"
 			(at 104.14 55.88 0)
 			(effects
@@
 			)
 		)
-		(property "Footprint" "0-moko_Library:CherryMX_Choc_Hotswap"
+		(property "Footprint" "0-moko_Library:CherryMX_Hotswap"
 			(at 127 35.56 0)
 			(effects
@@
 			)
 		)
-		(property "Footprint" "0-moko_Library:CherryMX_Choc_Hotswap"
+		(property "Footprint" "0-moko_Library:CherryMX_Hotswap"
 			(at 149.86 76.2 0)
 			(effects
@@
 			)
 		)
-		(property "Footprint" "0-moko_Library:CherryMX_Choc_Hotswap"
+		(property "Footprint" "0-moko_Library:CherryMX_Hotswap"
 			(at 125.73 165.1 0)
 			(effects
@@
 			)
 		)
-		(property "Footprint" "0-moko_Library:CherryMX_Choc_Hotswap"
+		(property "Footprint" "0-moko_Library:CherryMX_Hotswap"
 			(at 172.72 35.56 0)
 			(effects
