File: productfiles/circuitboard/moko/moko.kicad_pcb (KiCad board)
At the start: 2 copper layers, 39 parts, among them J1 Conn_01x06, J2 AudioJack4, J3 Conn_01x06, SW1 SW_Push, SW10 SW_Push, SW11 SW_Push, SW12 SW_Push, SW13 SW_Push, SW14 SW_Push, SW15 SW_Push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

Commit message: board upd8
Parts:
- RSW1: footprint 0-moko_Library:ResetSW_Anled_MJP1117 -> 0-moko_Library:ResetSW; moved to B.Cu
- SW1, SW10, SW11, SW12, SW13, SW14, SW15, SW16, SW17, SW2, SW3, SW4, SW5, SW6, SW7, SW8, SW9: footprint 0-moko_Library:CherryMX_Choc_Hotswap -> 0-moko_Library:CherryMX_Hotswap
- U1: footprint 0-moko_Library:ProMicro_v2 -> 0-moko_Library:ProMicro_rev_2
- moved D15 192.8 mm to (36.8, 116.4), turned to 90 degrees
- moved U1 191.0 mm to (29.7, 51.1)
- moved RSW1 185.9 mm to (28.2, 85.5), turned to 180 degrees
- moved SW15 175.5 mm to (28.5, 114.0)
- moved D10 162.9 mm to (57.6, 99.5)
- moved D11 162.9 mm to (57.6, 102.1)
- moved D12 162.9 mm to (57.6, 104.8)
- moved D4 162.9 mm to (51.0, 99.5)
- moved D5 162.9 mm to (51.0, 102.1)
- moved D6 162.9 mm to (51.0, 104.8)
- moved D9 162.9 mm to (57.6, 96.8)
- moved D16 162.9 mm to (64.1, 99.5)
- moved D17 162.9 mm to (64.1, 102.1)
- moved J1 162.9 mm to (49.0, 112.4)
- moved D1 160.1 mm to (55.8, 45.1), turned to 90 degrees
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Other:
- board outline added: 95 x 93.8 mm
